Commit message: ROS/diffdrive + camera working

File: verilator/poc_verilator_simulation/sim/example7/worlds/car1.0.urdf (robot description, URDF)
Before this commit: robot car, 4 links, 3 joints
Links:
- removed link base_link
- added link dummy
Joints:
- joint dummy_joint: parent base_link -> dummy
